Commit message: Changed the inertial tensor and mass of the body

File: urdf/sparkle.xacro (robot description, xacro)
@@ -1,10 +1,17 @@
 <?xml version="1.0"?>
 <robot name="$(arg roboname)" xmlns:xacro="http://www.ros.org/wiki/xacro">
- <xacro:property name="car_length" value="61.728100"/>
+ <!--xacro:property name="car_length" value="61.728100"/>
  <xacro:property name="car_width" value="157.523697"/>
  <xacro:property name="car_height" value="44.270203"/>
  <xacro:property name="scale_factor" value="0.0254"/>
  <xacro:property name="meshlab_factor" value="0.1"/>
- <xacro:property name="car_mass" value="10"/>
+ <xacro:property name="car_mass" value="1773.47881606"/>
+<xacro:property name="car_volume" value="433402.531250"/-->
+ <xacro:property name="car_length" value="4.00111"/>
+ <xacro:property name="car_width" value="2.13607648"/>
+ <xacro:property name="car_height" value="1.7"/>  <!-- This not Exact-->
+ <xacro:property name="scale_factor" value="0.7"/>
+ <xacro:property name="meshlab_factor" value="0.1"/>
+ <xacro:property name="car_mass" value="1773.47881606"/>
 <xacro:property name="car_volume" value="433402.531250"/>
 <xacro:property name="base_mass_ixx" value="1773.47881606"/>
@@ -20,5 +27,5 @@
 <link name="base_link">
       <collision name="collision">
-        <origin xyz="0 0 0" rpy="0 0 1.57079632679"/>
+        <origin xyz="0.0 0.0 0.0" rpy="0.0 0.0 1.57079632679"/>
         <geometry>
           <!--box size="${car_length*scale_factor} ${car_width*scale_factor} ${car_height*scale_factor}"/-->
@@ -27,5 +34,5 @@
       </collision>
       <visual name="visual">
-        <origin xyz="0 0 0" rpy="0 0 1.57079632679"/>
+        <origin xyz="0.0 0.0 0.0" rpy="0.0 0.0 1.57079632679"/>
         <geometry>
           <mesh scale="0.0254 0.0254 0.0254" filename="package://sparkle/meshes/hatchback.obj"/>
@@ -34,13 +41,14 @@
       <inertial>
                 <mass value="${car_mass}" />
-                <origin xyz="0 0 0" rpy="0 0 1.57079632679"/>
-                   <inertia
+                <!--origin xyz="0 0 ${car_height/2}" rpy="0 0 1.57079632679"/-->
+                <origin xyz="0.15 0.0 ${car_height*0.4}" rpy="0.0 0.0 0.0"/>
+                   <!--inertia
                 ixx="${base_mass_ixx}"  ixy="${base_mass_ixy}" ixz="${base_mass_ixz}"
                 iyx="${base_mass_iyx}" iyy="${base_mass_iyy}" iyz="${base_mass_iyz}"
-                izx="${base_mass_izx}" izy="${base_mass_izy}" izz="${base_mass_izz}"/>
-                <!--inertia ixx="${(1/6)*car_mass*( (car_width*scale_factor)*(car_width*scale_factor)  +   (car_height*scale_factor)*(car_height*scale_factor) )  }" ixy="0" ixz="0"
+                izx="${base_mass_izx}" izy="${base_mass_izy}" izz="${base_mass_izz}"/-->
+                <inertia ixx="${(1/6)*car_mass*( (car_width*scale_factor)*(car_width*scale_factor)  +   (car_height*scale_factor)*(car_height*scale_factor) )  }" ixy="0" ixz="0"
                 iyy="${(1/6)*car_mass*( (car_length*scale_factor)*(car_length*scale_factor)  +   (car_height*scale_factor)*(car_height*scale_factor) )  }" iyz="0"
                 izz="${(1/6)*car_mass*( (car_length*scale_factor)*(car_length*scale_factor)  +   (car_width*scale_factor)*(car_width*scale_factor) )  }" />
-                  <inertia ixx="${(1/6)*car_mass*( (car_width*scale_factor)*(car_width*scale_factor)  +   (car_height*scale_factor)*(car_height*scale_factor) )  }" ixy="0" ixz="0"
+                  <!--inertia ixx="${(1/6)*car_mass*( (car_width*scale_factor)*(car_width*scale_factor)  +   (car_height*scale_factor)*(car_height*scale_factor) )  }" ixy="0" ixz="0"
                 iyy="${(1/6)*car_mass*( (car_length*scale_factor)*(car_length*scale_factor)  +   (car_height*scale_factor)*(car_height*scale_factor) )  }" iyz="0"
                 izz="${(1/6)*car_mass*( (car_length*scale_factor)*(car_length*scale_factor)  +   (car_width*scale_factor)*(car_width*scale_factor) )  }" /-->

Commit message: Removed explicit tag for robot namespace. Plugin will use model's name as robot namespace

File: urdf/sparkle.xacro (robot description, xacro)
@@ -1,47 +1,95 @@
-<?xml version="1.0"?>
-<robot name="$(arg roboname)" xmlns:xacro="http://www.ros.org/wiki/xacro">
- <!--xacro:property name="car_length" value="61.728100"/>
- <xacro:property name="car_width" value="157.523697"/>
- <xacro:property name="car_height" value="44.270203"/>
- <xacro:property name="scale_factor" value="0.0254"/>
- <xacro:property name="meshlab_factor" value="0.1"/>
- <xacro:property name="car_mass" value="1773.47881606"/>
-<xacro:property name="car_volume" value="433402.531250"/-->
- <xacro:property name="car_length" value="4.00111"/>
- <xacro:property name="car_width" value="2.13607648"/>
- <xacro:property name="car_height" value="1.7"/>  <!-- This not Exact-->
- <xacro:property name="scale_factor" value="0.7"/>
- <xacro:property name="meshlab_factor" value="0.1"/>
- <xacro:property name="car_mass" value="1773.47881606"/>
-<xacro:property name="car_volume" value="433402.531250"/>
-<xacro:property name="base_mass_ixx" value="1773.47881606"/>
-    <xacro:property name="base_mass_ixy" value="0.00623522726"/>
-    <xacro:property name="base_mass_ixz" value="0.1256406519"/>
-    <xacro:property name="base_mass_iyx" value="0.00623522726"/>
-    <xacro:property name="base_mass_iyy" value="571.89989935"/>
-    <xacro:property name="base_mass_iyz" value="-115.176835391"/>
-    <xacro:property name="base_mass_izx" value="0.1256406519"/>
-    <xacro:property name="base_mass_izy" value="-115.176835391"/>
-    <xacro:property name="base_mass_izz" value="1974.56552349"/>
-<xacro:include filename="$(find sparkle)/urdf/sparkle.gazebo"/>
-<link name="base_link">
-      <collision name="collision">
-        <origin xyz="0.0 0.0 0.0" rpy="0.0 0.0 1.57079632679"/>
-        <geometry>
-          <!--box size="${car_length*scale_factor} ${car_width*scale_factor} ${car_height*scale_factor}"/-->
-          <mesh scale="0.0254 0.0254 0.0254" filename="package://sparkle/meshes/hatchback.obj"/>
-        </geometry>
-      </collision>
-      <visual name="visual">
-        <origin xyz="0.0 0.0 0.0" rpy="0.0 0.0 1.57079632679"/>
-        <geometry>
-          <mesh scale="0.0254 0.0254 0.0254" filename="package://sparkle/meshes/hatchback.obj"/>
-        </geometry>
-      </visual>
-      <inertial>
+<?xml version="1.0" ?>
+<!--
+Author: Rahul Bhadani, Jonathan Sprinkle, Rahul Bhadani
+Copyright (c) 2019-2020 Arizona Board of Regents
+All rights reserved.
+Permission is hereby granted, without written agreement and without
+license or royalty fees, to use, copy, modify, and distribute this
+software and its documentation for any purpose, provided that the
+above copyright notice and the following two paragraphs appear in
+all copies of this software.
+IN NO EVENT SHALL THE ARIZONA BOARD OF REGENTS BE LIABLE TO ANY PARTY
+FOR DIRECT, INDIRECT, SPECIAL, INCIDENTAL, OR CONSEQUENTIAL DAMAGES
+ARISING OUT OF THE USE OF THIS SOFTWARE AND ITS DOCUMENTATION, EVEN
+IF THE ARIZONA BOARD OF REGENTS HAS BEEN ADVISED OF THE POSSIBILITY OF
+SUCH DAMAGE.
+THE ARIZONA BOARD OF REGENTS SPECIFICALLY DISCLAIMS ANY WARRANTIES,
+    INCLUDING, BUT NOT LIMITED TO, THE IMPLIED WARRANTIES OF MERCHANTABILITY
+    AND FITNESS FOR A PARTICULAR PURPOSE. THE SOFTWARE PROVIDED HEREUNDER
+    IS ON AN "AS IS" BASIS, AND THE ARIZONA BOARD OF REGENTS HAS NO OBLIGATION
+    TO PROVIDE MAINTENANCE, SUPPORT, UPDATES, ENHANCEMENTS, OR MODIFICATIONS.
+    Summary:
+    =======
+    This file specifies 3D structure of the car with their inertial properties
+    and other dynamics.
+    -->
+    <robot name="$(arg roboname)" xmlns:xacro="http://www.ros.org/wiki/xacro">
+        <xacro:arg name="laser_sensor" default="false"/>
+        <xacro:property name="laser_sensor" value="$(arg laser_sensor)"/>
+        <xacro:property name="sensor_box" value="0.25"/>
+        <xacro:property name="PI" value="3.1415926835897931"/>
+        <xacro:property name="base_height" value="1.0639"/>
+        <xacro:property name="base_mass" value="1703.239"/>
+        <!-- car_to_bumper is car's length. The value reported here
+        is the lenght of the bounding box of the 3D mesh of the car's
+        body given by meshlab. Actual length of the car may be slightly
+        less and if require, we may use some offset to use this value
+        anywhere -->
+        <xacro:property name="car_to_bumper" value="4.25"/>
+        <!-- We are assuming that front bumper's height is half of the car's
+        bounding box height -->
+        <xacro:property name="front_bumper_height" value="${car_height/2}"/>
+        <!--This is the car tread, i.e distance between right and left front wheels-->
+        <xacro:property name="car_width_offset" value="0.05"/>
+        <xacro:property name="front_laser_size" value="0.25"/>
+        <xacro:property name="front_laser_mass" value="1"/>
+        <xacro:include filename="$(find sparkle)/urdf/sparkle.gazebo"/>
+        <xacro:arg name="laser_sensor" default="false"/>
+        <xacro:property name="laser_sensor" value="$(arg laser_sensor)"/>
+        <!--xacro:property name="car_length" value="61.728100"/>
+        <xacro:property name="car_width" value="157.523697"/>
+        <xacro:property name="car_height" value="44.270203"/>
+        <xacro:property name="scale_factor" value="0.0254"/>
+        <xacro:property name="meshlab_factor" value="0.1"/>
+        <xacro:property name="car_mass" value="1773.47881606"/>
+        <xacro:property name="car_volume" value="433402.531250"/-->
+        <xacro:property name="car_length" value="4.54"/>
+        <xacro:property name="car_width" value="1.79"/>
+        <xacro:property name="car_height" value="1.49"/>  <!-- This not Exact-->
+        <xacro:property name="scale_factor" value="0.88"/>
+        <xacro:property name="meshlab_factor" value="0.1"/>
+        <xacro:property name="car_mass" value="1800.0"/>
+        <xacro:property name="car_volume" value="433402.531250"/>
+        <xacro:property name="front_bumper_height" value="${car_height/3}"/>
+        <xacro:property name="base_mass_ixx" value="1773.47881606"/>
+        <xacro:property name="base_mass_ixy" value="0.00623522726"/>
+        <xacro:property name="base_mass_ixz" value="0.1256406519"/>
+        <xacro:property name="base_mass_iyx" value="0.00623522726"/>
+        <xacro:property name="base_mass_iyy" value="571.89989935"/>
+        <xacro:property name="base_mass_iyz" value="-115.176835391"/>
+        <xacro:property name="base_mass_izx" value="0.1256406519"/>
+        <xacro:property name="base_mass_izy" value="-115.176835391"/>
+        <xacro:property name="base_mass_izz" value="1974.56552349"/>
+        <xacro:property name="front_laser_size" value="0.25"/>
+        <xacro:property name="front_laser_mass" value="1.0"/>
+        <link name="base_link">
+            <collision name="collision">
+                <origin xyz="0.0 0.0 0.0" rpy="0.0 0.0 1.57079632679"/>
+                <geometry>
+                <!--box size="${car_length*scale_factor} ${car_width*scale_factor} ${car_height*scale_factor}"/-->
+                <mesh scale="0.01 0.01 0.01" filename="package://sparkle/meshes/Hybrid.obj"/>
+                </geometry>
+            </collision>
+            <visual name="visual">
+                <origin xyz="0.0 0.0 0.0" rpy="0.0 0.0 1.57079632679"/>
+                <geometry>
+                <mesh scale="0.01 0.01 0.01" filename="package://sparkle/meshes/Hybrid.obj"/>
+                </geometry>
+            </visual>
+            <inertial>
                 <mass value="${car_mass}" />
                 <!--origin xyz="0 0 ${car_height/2}" rpy="0 0 1.57079632679"/-->
-                <origin xyz="0.15 0.0 ${car_height*0.4}" rpy="0.0 0.0 0.0"/>
-                   <!--inertia
+                <origin xyz="0.0 0.0 0.0" rpy="0.0 0.0 0.0"/>
+                <!--inertia
                 ixx="${base_mass_ixx}"  ixy="${base_mass_ixy}" ixz="${base_mass_ixz}"
                 iyx="${base_mass_iyx}" iyy="${base_mass_iyy}" iyz="${base_mass_iyz}"
@@ -50,8 +98,44 @@
                 iyy="${(1/6)*car_mass*( (car_length*scale_factor)*(car_length*scale_factor)  +   (car_height*scale_factor)*(car_height*scale_factor) )  }" iyz="0"
                 izz="${(1/6)*car_mass*( (car_length*scale_factor)*(car_length*scale_factor)  +   (car_width*scale_factor)*(car_width*scale_factor) )  }" />
-                  <!--inertia ixx="${(1/6)*car_mass*( (car_width*scale_factor)*(car_width*scale_factor)  +   (car_height*scale_factor)*(car_height*scale_factor) )  }" ixy="0" ixz="0"
+                <!--inertia ixx="2581.13354740" ixy="0" ixz="0"
+                iyy="91.30846112" iyz="0"
+                izz="2681.95008628" /-->
+                <!--inertia ixx="${(1/6)*car_mass*( (car_width*scale_factor)*(car_width*scale_factor)  +   (car_height*scale_factor)*(car_height*scale_factor) )  }" ixy="0" ixz="0"
                 iyy="${(1/6)*car_mass*( (car_length*scale_factor)*(car_length*scale_factor)  +   (car_height*scale_factor)*(car_height*scale_factor) )  }" iyz="0"
                 izz="${(1/6)*car_mass*( (car_length*scale_factor)*(car_length*scale_factor)  +   (car_width*scale_factor)*(car_width*scale_factor) )  }" /-->
-    </inertial>
-</link>
-</robot>
+            </inertial>
+        </link>
+        <xacro:if value="$(arg laser_sensor)">
+            <xacro:include filename="$(find sparkle)/urdf/laser.gazebo"/>
+        <!-- front laser-->
+        <joint name="front_laser_joint" type="fixed">
+            <origin xyz="${car_to_bumper/2 + front_laser_size} 0 ${front_bumper_height + front_laser_size/2}" rpy="0 0 0"/>
+            <axis xyz="0 0 1"/>
+            <parent link="base_link"/>
+            <child link="front_laser_link"/>
+        </joint>
+        <link name="front_laser_link">
+            <parent link="front_laser_joint"/>
+            <collision>
+                <origin xyz="0 0 0" rpy="0 0.0 0"/>
+                <geometry>
+                <box size="${front_laser_size} ${front_laser_size} ${front_laser_size}"/>
+                </geometry>
+            </collision>
+            <visual>
+                <origin xyz="0 0 0" rpy="0 0 0"/>
+                <geometry>
+                <mesh filename="package://sparkle/meshes/SickLMS.dae"/>
+                <!--box size="${front_laser_size} ${front_laser_size} ${front_laser_size}"/-->
+                </geometry>
+            </visual>
+            <inertial>
+                <mass value="${front_laser_mass}" />
+                <origin xyz="0 0 0" rpy="0 0 0"/>
+                <inertia ixx="${(1/6)*front_laser_mass*front_laser_size*front_laser_size}" ixy="0" ixz="0"
+                iyy="${(1/6)*front_laser_mass*front_laser_size*front_laser_size}" iyz="0"
+                izz="${(1/6)*front_laser_mass*front_laser_size*front_laser_size}" />
+            </inertial>
+        </link>
+         </xacro:if>
+    </robot>
